File: ergo42_pcb_case/bottom/bottom.kicad_pcb (KiCad board)
At the start: 2 copper layers, 80.9 x 24.8 mm, 5 parts

Commit message: DXF -> KiCad -> plots
Parts:
- added REF**: MountingHole_2.2mm_M2_Pad, MountingHole_2.2mm_M2_Pad, F.Cu at (9.53, -9.53)
- added REF**: MountingHole_2.2mm_M2_Pad, MountingHole_2.2mm_M2_Pad, F.Cu at (104.8, -9.53)
- added REF**: MountingHole_2.2mm_M2_Pad, MountingHole_2.2mm_M2_Pad, F.Cu at (47.6, -28.6)
- added REF**: MountingHole_2.2mm_M2_Pad, MountingHole_2.2mm_M2_Pad, F.Cu at (9.53, -47.6)
- moved REF** 57.8 mm to (68.5, -91.0)
- moved REF** 56.6 mm to (104.8, -47.6)
- moved REF** 11.6 mm to (123.4, -73.0)
Other:
- board size 80.9 x 24.8 mm -> 139.2 x 106.9 mm
- rule pad_to_mask_clearance: 0.051 -> 0
Changed lines of the file:
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@@
   (general
     (thickness 1.6)
-    (drawings 13)
+    (drawings 21)
     (tracks 0)
     (zones 0)
-    (modules 5)
+    (modules 9)
     (nets 1)
   )
@@
     (uvia_min_size 0.2)
     (uvia_min_drill 0.1)
-    (edge_width 0.05)
+    (edge_width 0.1)
     (segment_width 0.2)
     (pcb_text_width 0.3)
     (pcb_text_size 1.5 1.5)
-    (mod_edge_width 0.12)
+    (mod_edge_width 0.15)
     (mod_text_size 1 1)
     (mod_text_width 0.15)
     (pad_size 1.524 1.524)
     (pad_drill 0.762)
-    (pad_to_mask_clearance 0.051)
-    (solder_mask_min_width 0.25)
+    (pad_to_mask_clearance 0)
     (aux_axis_origin 0 0)
     (visible_elements FFFFFF7F)
@@
   )
   (module MountingHole_2.2mm_M2_Pad (layer F.Cu)
-    (at 111.76 -73.025)
+    (at 9.525 -9.525)
+    (descr "Mounting Hole 2.2mm, M2")
+    (tags "mounting hole 2.2mm m2")
+    (attr virtual)
+    (fp_text reference REF** (at 0 -3.2) (layer F.SilkS) hide
+      (effects (font (size 1 1) (thickness 0.15)))
+    )
+    (fp_text value MountingHole_2.2mm_M2_Pad (at 0 3.2) (layer F.Fab)
+      (effects (font (size 1 1) (thickness 0.15)))
+    )
+    (fp_circle (center 0 0) (end 2.45 0) (layer F.CrtYd) (width 0.05))
+    (fp_circle (center 0 0) (end 2.2 0) (layer Cmts.User) (width 0.15))
+    (fp_text user %R (at 0.3 0) (layer F.Fab)
+      (effects (font (size 1 1) (thickness 0.15)))
+    )
+    (pad 1 thru_hole circle (at 0 0) (size 4.4 4.4) (drill 2.2) (layers *.Cu *.Mask))
+  )
+  (module MountingHole_2.2mm_M2_Pad (layer F.Cu)
+    (at 104.775 -9.525)
+    (descr "Mounting Hole 2.2mm, M2")
+    (tags "mounting hole 2.2mm m2")
+    (attr virtual)
+    (fp_text reference REF** (at 0 -3.2) (layer F.SilkS) hide
+      (effects (font (size 1 1) (thickness 0.15)))
+    )
+    (fp_text value MountingHole_2.2mm_M2_Pad (at 0 3.2) (layer F.Fab)
+      (effects (font (size 1 1) (thickness 0.15)))
+    )
+    (fp_circle (center 0 0) (end 2.45 0) (layer F.CrtYd) (width 0.05))
+    (fp_circle (center 0 0) (end 2.2 0) (layer Cmts.User) (width 0.15))
+    (fp_text user %R (at 0.3 0) (layer F.Fab)
+      (effects (font (size 1 1) (thickness 0.15)))
+    )
+    (pad 1 thru_hole circle (at 0 0) (size 4.4 4.4) (drill 2.2) (layers *.Cu *.Mask))
+  )
+  (module MountingHole_2.2mm_M2_Pad (layer F.Cu)
+    (at 47.625 -28.575)
+    (descr "Mounting Hole 2.2mm, M2")
+    (tags "mounting hole 2.2mm m2")
+    (attr virtual)
+    (fp_text reference REF** (at 0 -3.2) (layer F.SilkS) hide
+      (effects (font (size 1 1) (thickness 0.15)))
+    )
+    (fp_text value MountingHole_2.2mm_M2_Pad (at 0 3.2) (layer F.Fab)
+      (effects (font (size 1 1) (thickness 0.15)))
+    )
+    (fp_circle (center 0 0) (end 2.45 0) (layer F.CrtYd) (width 0.05))
+    (fp_circle (center 0 0) (end 2.2 0) (layer Cmts.User) (width 0.15))
+    (fp_text user %R (at 0.3 0) (layer F.Fab)
+      (effects (font (size 1 1) (thickness 0.15)))
+    )
+    (pad 1 thru_hole circle (at 0 0) (size 4.4 4.4) (drill 2.2) (layers *.Cu *.Mask))
+  )
+  (module MountingHole_2.2mm_M2_Pad (layer F.Cu)
+    (at 9.525 -47.625)
+    (descr "Mounting Hole 2.2mm, M2")
+    (tags "mounting hole 2.2mm m2")
+    (attr virtual)
+    (fp_text reference REF** (at 0 -3.2) (layer F.SilkS) hide
+      (effects (font (size 1 1) (thickness 0.15)))
+    )
+    (fp_text value MountingHole_2.2mm_M2_Pad (at 0 3.2) (layer F.Fab)
+      (effects (font (size 1 1) (thickness 0.15)))
+    )
+    (fp_circle (center 0 0) (end 2.45 0) (layer F.CrtYd) (width 0.05))
+    (fp_circle (center 0 0) (end 2.2 0) (layer Cmts.User) (width 0.15))
+    (fp_text user %R (at 0.3 0) (layer F.Fab)
+      (effects (font (size 1 1) (thickness 0.15)))
+    )
+    (pad 1 thru_hole circle (at 0 0) (size 4.4 4.4) (drill 2.2) (layers *.Cu *.Mask))
+  )
+  (module MountingHole_2.2mm_M2_Pad (layer F.Cu)
+    (at 123.395 -73.005)
     (descr "Mounting Hole 2.2mm, M2")
     (tags "mounting hole 2.2mm m2")
@@
   )
   (module MountingHole_2.2mm_M2_Pad (layer F.Cu)
-    (at 123.395 -73.005)
+    (at 68.494507 -91.01)
     (descr "Mounting Hole 2.2mm, M2")
     (tags "mounting hole 2.2mm m2")
@@
   )
   (module MountingHole_2.2mm_M2_Pad (layer F.Cu)
-    (at 68.494507 -91.01)
-    (descr "Mounting Hole 2.2mm, M2")
-    (tags "mounting hole 2.2mm m2")
-    (attr virtual)
-    (fp_text reference REF** (at 0 -3.2) (layer F.SilkS) hide
-      (effects (font (size 1 1) (thickness 0.15)))
-    )
-    (fp_text value MountingHole_2.2mm_M2_Pad (at 0 3.2) (layer F.Fab)
-      (effects (font (size 1 1) (thickness 0.15)))
-    )
-    (fp_circle (center 0 0) (end 2.45 0) (layer F.CrtYd) (width 0.05))
-    (fp_circle (center 0 0) (end 2.2 0) (layer Cmts.User) (width 0.15))
-    (fp_text user %R (at 0.3 0) (layer F.Fab)
-      (effects (font (size 1 1) (thickness 0.15)))
-    )
-    (pad 1 thru_hole circle (at 0 0) (size 4.4 4.4) (drill 2.2) (layers *.Cu *.Mask))
-  )
+    (at 104.775 -47.625)
+    (descr "Mounting Hole 2.2mm, M2")
+    (tags "mounting hole 2.2mm m2")
+    (attr virtual)
+    (fp_text reference REF** (at 0 -3.2) (layer F.SilkS) hide
+      (effects (font (size 1 1) (thickness 0.15)))
+    )
+    (fp_text value MountingHole_2.2mm_M2_Pad (at 0 3.2) (layer F.Fab)
+      (effects (font (size 1 1) (thickness 0.15)))
+    )
+    (fp_circle (center 0 0) (end 2.45 0) (layer F.CrtYd) (width 0.05))
+    (fp_circle (center 0 0) (end 2.2 0) (layer Cmts.User) (width 0.15))
+    (fp_text user %R (at 0.3 0) (layer F.Fab)
+      (effects (font (size 1 1) (thickness 0.15)))
+    )
+    (pad 1 thru_hole circle (at 0 0) (size 4.4 4.4) (drill 2.2) (layers *.Cu *.Mask))
+  )
+  (gr_circle (center 104.775 -47.625) (end 105.95 -47.625) (layer Eco1.User) (width 0.2))
+  (gr_circle (center 50.489507 -73.005) (end 51.664507 -73.005) (layer Eco1.User) (width 0.2))
   (gr_circle (center 68.494507 -91.01) (end 69.669507 -91.01) (layer Eco1.User) (width 0.2))
-  (gr_circle (center 50.489507 -73.005) (end 51.664507 -73.005) (layer Eco1.User) (width 0.2))
+  (gr_circle (center 123.395 -91.01) (end 124.57 -91.01) (layer Eco1.User) (width 0.2))
   (gr_circle (center 123.395 -73.005) (end 124.57 -73.005) (layer Eco1.User) (width 0.2))
-  (gr_circle (center 123.395 -91.01) (end 124.57 -91.01) (layer Eco1.User) (width 0.2))
-  (gr_circle (center 111.76 -73.025) (end 112.935 -73.025) (layer Eco1.User) (width 0.2))
-  (gr_arc (start 48.364999 -72.125) (end 46.597233 -73.892766) (angle -135) (layer Edge.Cuts) (width 0.2))
-  (gr_line (start 124.274999 -69.625) (end 48.364999 -69.625) (layer Edge.Cuts) (width 0.2))
-  (gr_arc (start 124.274999 -72.125) (end 124.274999 -69.625) (angle -90) (layer Edge.Cuts) (width 0.2))
-  (gr_line (start 126.774999 -91.889999) (end 126.774999 -72.125) (layer Edge.Cuts) (width 0.2))
-  (gr_arc (start 124.274999 -91.889999) (end 126.774999 -91.889999) (angle -90) (layer Edge.Cuts) (width 0.2))
-  (gr_line (start 68.129999 -94.39) (end 124.274999 -94.389999) (layer Edge.Cuts) (width 0.2))
-  (gr_arc (start 68.129999 -91.89) (end 68.129999 -94.39) (angle -45) (layer Edge.Cuts) (width 0.2))
-  (gr_line (start 46.597233 -73.892766) (end 66.362233 -93.657766) (layer Edge.Cuts) (width 0.2))
+  (gr_circle (center 9.525 -47.625) (end 10.7 -47.625) (layer Eco1.User) (width 0.2))
+  (gr_circle (center 47.625 -28.575) (end 48.8 -28.575) (layer Eco1.User) (width 0.2))
+  (gr_circle (center 104.775 -9.525) (end 105.95 -9.525) (layer Eco1.User) (width 0.2))
+  (gr_circle (center 9.525 -9.525) (end 10.7 -9.525) (layer Eco1.User) (width 0.2))
+  (gr_arc (start -9.975 9.975) (end -12.475 9.975) (angle -90) (layer Edge.Cuts) (width 0.2))
+  (gr_line (start 124.275 12.475) (end -9.975 12.475) (layer Edge.Cuts) (width 0.2))
+  (gr_arc (start 124.275 9.975) (end 124.275 12.475) (angle -90) (layer Edge.Cuts) (width 0.2))
+  (gr_line (start 126.775 -91.889999) (end 126.775 9.974999) (layer Edge.Cuts) (width 0.2))
+  (gr_arc (start 124.275 -91.889999) (end 126.775 -91.889999) (angle -90) (layer Edge.Cuts) (width 0.2))
+  (gr_line (start 68.129999 -94.389999) (end 124.275 -94.389999) (layer Edge.Cuts) (width 0.2))
+  (gr_arc (start 68.129999 -91.889999) (end 68.129999 -94.389999) (angle -45) (layer Edge.Cuts) (width 0.2))
+  (gr_line (start 43.061699 -70.357233) (end 66.362233 -93.657766) (layer Edge.Cuts) (width 0.2))
+  (gr_arc (start 41.293932 -72.125) (end 41.293932 -69.625) (angle -45) (layer Edge.Cuts) (width 0.2))
+  (gr_line (start -9.975 -69.625) (end 41.293932 -69.625) (layer Edge.Cuts) (width 0.2))
+  (gr_arc (start -9.975 -67.125) (end -9.975 -69.625) (angle -90) (layer Edge.Cuts) (width 0.2))
+  (gr_line (start -12.475 9.974999) (end -12.475 -67.125) (layer Edge.Cuts) (width 0.2))
 )

Commit message: Reimport DXFs into middle of the page
PDF plotter has hard times with anything outside A4 page...
Parts:
- removed the REF** at (9.53, -9.53)
- removed the REF** at (104.8, -9.53)
- removed the REF** at (47.6, -28.6)
- removed the REF** at (9.53, -47.6)
- removed the REF** at (123.4, -73.0)
- removed the REF** at (123.4, -91.0)
- removed the REF** at (68.5, -91.0)
- removed the REF** at (50.5, -73.0)
- removed the REF** at (104.8, -47.6)
- added REF**: MountingHole_2.2mm_M2_Pad, MountingHole_2.2mm_M2_Pad, F.Cu at (208.8, 47.8)
- added REF**: MountingHole_2.2mm_M2_Pad, MountingHole_2.2mm_M2_Pad, F.Cu at (153.9, 47.8)
- added REF**: MountingHole_2.2mm_M2_Pad, MountingHole_2.2mm_M2_Pad, F.Cu at (190.2, 129.3)
- added REF**: MountingHole_2.2mm_M2_Pad, MountingHole_2.2mm_M2_Pad, F.Cu at (133.0, 110.3)
- added REF**: MountingHole_2.2mm_M2_Pad, MountingHole_2.2mm_M2_Pad, F.Cu at (94.9, 91.2)
- added REF**: MountingHole_2.2mm_M2_Pad, MountingHole_2.2mm_M2_Pad, F.Cu at (135.9, 65.8)
- added REF**: MountingHole_2.2mm_M2_Pad, MountingHole_2.2mm_M2_Pad, F.Cu at (190.2, 91.2)
- added REF**: MountingHole_2.2mm_M2_Pad, MountingHole_2.2mm_M2_Pad, F.Cu at (208.8, 65.8)
- added REF**: MountingHole_2.2mm_M2_Pad, MountingHole_2.2mm_M2_Pad, F.Cu at (94.9, 129.3)
Other:
- board size 139.2 x 106.9 mm -> 139.3 x 106.9 mm
Changed lines of the file:
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@@
   )
   (module MountingHole_2.2mm_M2_Pad (layer F.Cu)
-    (at 9.525 -9.525)
+    (at 208.78 47.84)
     (descr "Mounting Hole 2.2mm, M2")
     (tags "mounting hole 2.2mm m2")
@@
   )
   (module MountingHole_2.2mm_M2_Pad (layer F.Cu)
-    (at 104.775 -9.525)
+    (at 153.879507 47.84)
     (descr "Mounting Hole 2.2mm, M2")
     (tags "mounting hole 2.2mm m2")
@@
   )
   (module MountingHole_2.2mm_M2_Pad (layer F.Cu)
-    (at 47.625 -28.575)
+    (at 190.16 129.325)
     (descr "Mounting Hole 2.2mm, M2")
     (tags "mounting hole 2.2mm m2")
@@
   )
   (module MountingHole_2.2mm_M2_Pad (layer F.Cu)
-    (at 9.525 -47.625)
+    (at 133.01 110.275)
     (descr "Mounting Hole 2.2mm, M2")
     (tags "mounting hole 2.2mm m2")
@@
   )
   (module MountingHole_2.2mm_M2_Pad (layer F.Cu)
-    (at 123.395 -73.005)
+    (at 94.91 91.225)
     (descr "Mounting Hole 2.2mm, M2")
     (tags "mounting hole 2.2mm m2")
@@
   )
   (module MountingHole_2.2mm_M2_Pad (layer F.Cu)
-    (at 123.395 -91.01)
+    (at 135.874507 65.845)
     (descr "Mounting Hole 2.2mm, M2")
     (tags "mounting hole 2.2mm m2")
@@
   )
   (module MountingHole_2.2mm_M2_Pad (layer F.Cu)
-    (at 68.494507 -91.01)
+    (at 190.16 91.225)
     (descr "Mounting Hole 2.2mm, M2")
     (tags "mounting hole 2.2mm m2")
@@
   )
   (module MountingHole_2.2mm_M2_Pad (layer F.Cu)
-    (at 50.489507 -73.005)
+    (at 208.78 65.845)
     (descr "Mounting Hole 2.2mm, M2")
     (tags "mounting hole 2.2mm m2")
@@
   )
   (module MountingHole_2.2mm_M2_Pad (layer F.Cu)
-    (at 104.775 -47.625)
+    (at 94.91 129.325)
     (descr "Mounting Hole 2.2mm, M2")
     (tags "mounting hole 2.2mm m2")
@@
     (pad 1 thru_hole circle (at 0 0) (size 4.4 4.4) (drill 2.2) (layers *.Cu *.Mask))
   )
-  (gr_circle (center 104.775 -47.625) (end 105.95 -47.625) (layer Eco1.User) (width 0.2))
-  (gr_circle (center 50.489507 -73.005) (end 51.664507 -73.005) (layer Eco1.User) (width 0.2))
-  (gr_circle (center 68.494507 -91.01) (end 69.669507 -91.01) (layer Eco1.User) (width 0.2))
-  (gr_circle (center 123.395 -91.01) (end 124.57 -91.01) (layer Eco1.User) (width 0.2))
-  (gr_circle (center 123.395 -73.005) (end 124.57 -73.005) (layer Eco1.User) (width 0.2))
-  (gr_circle (center 9.525 -47.625) (end 10.7 -47.625) (layer Eco1.User) (width 0.2))
-  (gr_circle (center 47.625 -28.575) (end 48.8 -28.575) (layer Eco1.User) (width 0.2))
-  (gr_circle (center 104.775 -9.525) (end 105.95 -9.525) (layer Eco1.User) (width 0.2))
-  (gr_circle (center 9.525 -9.525) (end 10.7 -9.525) (layer Eco1.User) (width 0.2))
-  (gr_arc (start -9.975 9.975) (end -12.475 9.975) (angle -90) (layer Edge.Cuts) (width 0.2))
-  (gr_line (start 124.275 12.475) (end -9.975 12.475) (layer Edge.Cuts) (width 0.2))
-  (gr_arc (start 124.275 9.975) (end 124.275 12.475) (angle -90) (layer Edge.Cuts) (width 0.2))
-  (gr_line (start 126.775 -91.889999) (end 126.775 9.974999) (layer Edge.Cuts) (width 0.2))
-  (gr_arc (start 124.275 -91.889999) (end 126.775 -91.889999) (angle -90) (layer Edge.Cuts) (width 0.2))
-  (gr_line (start 68.129999 -94.389999) (end 124.275 -94.389999) (layer Edge.Cuts) (width 0.2))
-  (gr_arc (start 68.129999 -91.889999) (end 68.129999 -94.389999) (angle -45) (layer Edge.Cuts) (width 0.2))
-  (gr_line (start 43.061699 -70.357233) (end 66.362233 -93.657766) (layer Edge.Cuts) (width 0.2))
-  (gr_arc (start 41.293932 -72.125) (end 41.293932 -69.625) (angle -45) (layer Edge.Cuts) (width 0.2))
-  (gr_line (start -9.975 -69.625) (end 41.293932 -69.625) (layer Edge.Cuts) (width 0.2))
-  (gr_arc (start -9.975 -67.125) (end -9.975 -69.625) (angle -90) (layer Edge.Cuts) (width 0.2))
-  (gr_line (start -12.475 9.974999) (end -12.475 -67.125) (layer Edge.Cuts) (width 0.2))
+  (gr_circle (center 94.91 129.325) (end 96.085 129.325) (layer Eco1.User) (width 0.2))
+  (gr_line (start 212.16 46.960001) (end 212.16 148.824999) (layer Edge.Cuts) (width 0.2))
+  (gr_circle (center 208.78 65.845) (end 209.955 65.845) (layer Eco1.User) (width 0.2))
+  (gr_arc (start 126.678932 66.725) (end 126.678932 69.225) (angle -45) (layer Edge.Cuts) (width 0.2))
+  (gr_line (start 209.66 151.325) (end 75.409999 151.325) (layer Edge.Cuts) (width 0.2))
+  (gr_circle (center 190.16 91.225) (end 191.335 91.225) (layer Eco1.User) (width 0.2))
+  (gr_arc (start 209.66 148.825) (end 209.66 151.325) (angle -90) (layer Edge.Cuts) (width 0.2))
+  (gr_circle (center 135.874507 65.845) (end 137.049507 65.845) (layer Eco1.User) (width 0.2))
+  (gr_line (start 75.409999 69.225) (end 126.678932 69.225) (layer Edge.Cuts) (width 0.2))
+  (gr_arc (start 209.66 46.960001) (end 212.16 46.960001) (angle -90) (layer Edge.Cuts) (width 0.2))
+  (gr_arc (start 75.409999 148.825) (end 72.909999 148.825) (angle -90) (layer Edge.Cuts) (width 0.2))
+  (gr_circle (center 94.91 91.225) (end 96.085 91.225) (layer Eco1.User) (width 0.2))
+  (gr_circle (center 133.01 110.275) (end 134.185 110.275) (layer Eco1.User) (width 0.2))
+  (gr_line (start 153.515 44.460001) (end 209.66 44.460001) (layer Edge.Cuts) (width 0.2))
+  (gr_circle (center 190.16 129.325) (end 191.335 129.325) (layer Eco1.User) (width 0.2))
+  (gr_line (start 72.909999 148.824999) (end 72.909999 71.725) (layer Edge.Cuts) (width 0.2))
+  (gr_circle (center 153.879507 47.84) (end 155.054507 47.84) (layer Eco1.User) (width 0.2))
+  (gr_line (start 128.446699 68.492767) (end 151.747233 45.192234) (layer Edge.Cuts) (width 0.2))
+  (gr_arc (start 75.409999 71.725) (end 75.409999 69.225) (angle -90) (layer Edge.Cuts) (width 0.2))
+  (gr_arc (start 153.515 46.960001) (end 153.515 44.460001) (angle -45) (layer Edge.Cuts) (width 0.2))
+  (gr_circle (center 208.78 47.84) (end 209.955 47.84) (layer Eco1.User) (width 0.2))
 )
